Commit message: urdf update. mobile_base_body_link should deprecate mobile_base_body

File: app/iKartRos/model/ikart.urdf (robot description, URDF)
Before this commit: robot ikart, 3 links, 2 joints
Links:
- added link mobile_base_body_link
Joints:
- added joint base_joint2: type fixed, parent mobile_base_body, child mobile_base_body_link, origin xyz=0 0.0 0.0   rpy=0 0 0

Commit message: ikart ROS navigation update

File: app/iKartRos/model/ikart.urdf (robot description, URDF)
Before this commit: robot ikart, 4 links, 3 joints
Links:
- added link base_laser
Joints:
- added joint laser_joint2: type fixed, parent mobile_base_body, child base_laser, origin xyz=0 0 0   rpy=0 0 0
